Commit message: Driving in sim - gazebo

File: pc/src/salamanca/description/robot.urdf.xacro (robot description, xacro)
@@ -3,3 +3,4 @@
     <xacro:include filename="common_properties.xacro" />
     <xacro:include filename="robot_core.xacro"/>
+    <xacro:include filename="gazebo_control.xacro"/>
 </robot>

File: pc/src/salamanca/description/robot_core.xacro (robot description, xacro)
@@ -47,11 +47,11 @@
         <visual>
             <geometry>
-                <mesh filename="package://salamanca/meshes/base_link.stl" scale="${scale_factor} ${scale_factor} ${scale_factor}" />
+                <box size="${base_length} ${base_width} ${base_height}" />
             </geometry>
             <origin xyz="0 0 0" rpy="0 0 0" />
         </visual>
-         <collision>
+        <collision>
             <geometry>
-                <mesh filename="package://salamanca/meshes/base_link.stl" scale="${scale_factor} ${scale_factor} ${scale_factor}" />
+                <box size="${base_length} ${base_width} ${base_height}" />
             </geometry>
             <origin xyz="0 0 0" rpy="0 0 0" />
@@ -60,4 +60,7 @@
             xyz="0 0 0" rpy="0 0 0" />
     </link>
+    <gazebo reference="platform">
+        <material>Gazebo/Black</material>
+    </gazebo>
     <!-- Left wheel link -->
     <joint name="left_wheel_joint" type="continuous">
@@ -82,4 +85,7 @@
             xyz="0 0 0" rpy="0 0 0" />
     </link>
+    <gazebo reference="left_wheel">
+        <material>Gazebo/Grey</material>
+    </gazebo>
     <!-- Right wheel link -->
     <joint name="right_wheel_joint" type="continuous">
@@ -104,19 +110,22 @@
             xyz="0 0 0" rpy="0 0 0" />
     </link>
+    <gazebo reference="right_wheel">
+        <material>Gazebo/Grey</material>
+    </gazebo>
     <!-- Castor Wheel link -->
     <joint name="castor_joint" type="fixed">
         <parent link="base_link" />
         <child link="castor_wheel" />
-        <origin xyz="${-(2/7)*base_length + 0.01} 0 ${odrive_radius}" rpy="0 0 0" />
+        <origin xyz="${-(2/7)*base_length + 0.01} 0 ${odrive_radius/2}" rpy="0 0 0" />
     </joint>
     <link name="castor_wheel">
         <visual>
             <geometry>
-                <mesh filename="package://salamanca/meshes/castor_wheel.stl" scale="${scale_factor} ${scale_factor} ${scale_factor}" />
+                <sphere radius="${odrive_radius/2}" />
             </geometry>
         </visual>
         <collision>
             <geometry>
-                <mesh filename="package://salamanca/meshes/castor_wheel.stl" scale="${scale_factor} ${scale_factor} ${scale_factor}" />
+                <sphere radius="${odrive_radius/2}" />
             </geometry>
             <origin xyz="0 0 0" rpy="0 0 0" />
@@ -125,3 +134,8 @@
             xyz="0 0 0" rpy="0 0 0" />
     </link>
+    <gazebo reference="castor_wheel">
+        <material>Gazebo/Grey</material>
+        <mu1 value="0.001"/>
+        <mu2 value="0.001"/>
+    </gazebo>
 </robot>

Commit message: Camera - gazebo

File: pc/src/salamanca/description/robot.urdf.xacro (robot description, xacro)
@@ -4,3 +4,5 @@
     <xacro:include filename="robot_core.xacro"/>
     <xacro:include filename="gazebo_control.xacro"/>
+    <xacro:include filename="lidar.xacro"/>
+    <xacro:include filename="camera.xacro"/>
 </robot>

File: pc/src/salamanca/description/robot_core.xacro (robot description, xacro)
@@ -12,6 +12,6 @@
     <xacro:property name="castor_mass" value="0.08" />
     <!--Realsense size -->
-    <xacro:property name="realsense_length" value="0.09" />
-    <xacro:property name="realsense_width" value="0.025" />
+    <xacro:property name="realsense_length" value="0.025" />
+    <xacro:property name="realsense_width" value="0.09" />
     <xacro:property name="realsense_height" value="0.025" />
     <xacro:property name="realsense_mass" value="0.072" />
@@ -21,6 +21,5 @@
     <xacro:property name="jetson_height" value="0.029" />
     <xacro:property name="jetson_mass" value="0.28" />
-    <!--Odrive size
-    (TODO: set teh correct dimensions)-->
+    <!--Odrive size -->
     <xacro:property name="odrive_radius" value="0.0855" />
     <xacro:property name="odrive_height" value="0.045" />
@@ -62,4 +61,29 @@
     <gazebo reference="platform">
         <material>Gazebo/Black</material>
+    </gazebo>
+    <!-- Battery link -->
+    <joint name="battery_joint" type="fixed">
+        <parent link="platform" />
+        <child link="battery" />
+        <origin xyz="-0.08 0 ${battery_height/2}" rpy="0 0 0" />
+    </joint>
+    <link name="battery">
+        <visual>
+            <geometry>
+                <box size="${battery_length} ${battery_width} ${battery_height}" />
+            </geometry>
+            <origin xyz="0 0 0" rpy="0 0 0" />
+        </visual>
+        <collision>
+            <geometry>
+                <box size="${battery_length} ${battery_width} ${battery_height}" />
+            </geometry>
+            <origin xyz="0 0 0" rpy="0 0 0" />
+        </collision>
+        <xacro:box_inertia m="${battery_mass}" l="${battery_length}" w="${battery_width}" h="${battery_height}"
+            xyz="0 0 0" rpy="0 0 0" />
+    </link>
+    <gazebo reference="battery">
+        <material>Gazebo/Grey</material>
     </gazebo>
     <!-- Left wheel link -->
